File: hw/i4screenhsmc.brd (EAGLE design)
At the start: 127 x 78.1 mm, 67 parts, among them CON1 IPHONE4_LCD_CONN, J1 QTH-090-XX-X-D-A, Q6 BSS84, U1 TPS622XX, U2 TPS622XX

Commit message: the N-channel FET is a BSS138, not a BSS84 (which is P-channel)
Parts:
- Q6: value BSS84 -> BSS138
Changed lines of the file:
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@@
 <?xml version="1.0" encoding="utf-8"?>
 <!DOCTYPE eagle SYSTEM "eagle.dtd">
-<eagle version="6.5.0">
+<eagle version="6.6.0">
 <drawing>
 <settings>
@@
 <attribute name="VALUE" x="80.71" y="4.02" size="1.27" layer="27" rot="R270"/>
 </element>
-<element name="Q6" library="SparkFun" package="SOT23-3" value="BSS84" x="85.5" y="5.75" smashed="yes" rot="MR180">
+<element name="Q6" library="SparkFun" package="SOT23-3" value="BSS138" x="85.5" y="5.75" smashed="yes" rot="MR180">
 <attribute name="NAME" x="87.376" y="4.572" size="1.016" layer="26" ratio="10" rot="MR270"/>
 <attribute name="VALUE" x="84.484" y="5.9405" size="0.4064" layer="28" rot="MR180"/>
